Commit message: make compliant with one-step launch script, add documentation

File: src/nautilus_description/urdf/nautilus.urdf (robot description, URDF)
Before this commit: robot nautilus, 9 links, 8 joints
Joints:
- joint motor_A_joint: origin xyz=0.16 -0.34 -0.02 rpy=-1.5707963267948966 0.0 -0.7853981633974483 -> xyz=0.16 -0.34 -0.02 rpy=1.5707963267948966 0.0 -0.7853981633974483
- joint motor_B_joint: origin xyz=-0.16 -0.34 -0.02 rpy=-1.5707963267948966 0.0 0.7853981633974483 -> xyz=-0.16 -0.34 -0.02 rpy=1.5707963267948966 0.0 0.7853981633974483
- joint motor_C_joint: origin xyz=0.16 0.07 -0.02 rpy=-1.5707963267948966 0.0 0.7853981633974483 -> xyz=0.16 0.07 -0.02 rpy=1.5707963267948966 0.0 0.7853981633974483
- joint motor_D_joint: origin xyz=-0.16 0.07 -0.02 rpy=-1.5707963267948966 0.0 -0.7853981633974483 -> xyz=-0.16 0.07 -0.02 rpy=1.5707963267948966 0.0 -0.7853981633974483
- joint motor_E_joint: origin xyz=0.165 -0.135 -0.02 rpy=3.141592653589793 0.0 0.0 -> xyz=0.165 -0.135 -0.02 rpy=0.0 0.0 0.0
- joint motor_F_joint: origin xyz=-0.165 -0.135 -0.02 rpy=3.141592653589793 0.0 0.0 -> xyz=-0.165 -0.135 -0.02 rpy=0.0 0.0 0.0

File: src/nautilus_description/urdf/nautilus.urdf.xacro (robot description, xacro)
@@ -81,10 +81,10 @@
   <!-- y+ -> back -->
   <!-- z+ -> up -->
-  <xacro:thrusters thrusterName="motor_A" x=".16" y="-.34" z="-.02" r="-${pi/2}" p="0.0" yaw="-${pi/4}"/>
-  <xacro:thrusters thrusterName="motor_B" x="-.16" y="-.34" z="-.02" r="-${pi/2}" p="0.0" yaw="${pi/4}"/>
-  <xacro:thrusters thrusterName="motor_C" x=".16" y=".07" z="-.02" r="-${pi/2}" p="0.0" yaw="${pi/4}"/>
-  <xacro:thrusters thrusterName="motor_D" x="-.16" y=".07" z="-.02" r="-${pi/2}" p="0.0" yaw="-${pi/4}"/>
-  <xacro:thrusters thrusterName="motor_E" x=".165" y="-.135" z="-.02" r="${pi}" p="0.0" yaw="0.0"/>
-  <xacro:thrusters thrusterName="motor_F" x="-.165" y="-.135" z="-.02" r="${pi}" p="0.0" yaw="0.0"/>
+  <xacro:thrusters thrusterName="motor_A" x=".16" y="-.34" z="-.02" r="${pi/2}" p="0.0" yaw="-${pi/4}"/>
+  <xacro:thrusters thrusterName="motor_B" x="-.16" y="-.34" z="-.02" r="${pi/2}" p="0.0" yaw="${pi/4}"/>
+  <xacro:thrusters thrusterName="motor_C" x=".16" y=".07" z="-.02" r="${pi/2}" p="0.0" yaw="${pi/4}"/>
+  <xacro:thrusters thrusterName="motor_D" x="-.16" y=".07" z="-.02" r="${pi/2}" p="0.0" yaw="-${pi/4}"/>
+  <xacro:thrusters thrusterName="motor_E" x=".165" y="-.135" z="-.02" r="0.0" p="0.0" yaw="0.0"/>
+  <xacro:thrusters thrusterName="motor_F" x="-.165" y="-.135" z="-.02" r="0.0" p="0.0" yaw="0.0"/>
   <xacro:cameras cameraName="camera1" x="0.0" y="-0.32" z="0.0" r="0.0" p="0.0" yaw="0.0"/>
   <xacro:cameras cameraName="camera2" x="0.0" y="-0.20" z="-.125" r="0.0" p="0.0" yaw="0.0"/>

Commit message: Imported dummy model, fixed main body mass, not neutral yet

File: src/nautilus_description/urdf/nautilus.urdf (robot description, URDF)
Before this commit: robot nautilus, 9 links, 8 joints
Links:
- link body: mass 21.576 -> 60.177; geometry collision mesh filename=model://nautilus/meshes/nautilus_sim.dae; visual mesh filename=model://nautilus/meshes/nautilus_sim.dae

File: src/nautilus_description/urdf/nautilus.urdf.xacro (robot description, xacro)
@@ -12,18 +12,18 @@
   <link name="body">
     <inertial>
-      <origin xyz="0.0 -.135 0.0" rpy="0.0 0.0 0.0"/>
+      <origin xyz="0 0 0" rpy="0.0 0.0 0.0"/>
       <!-- TOOD: get a better mass estimate -->
-      <mass value="21.576"/>
+      <mass value="60.177"/>
      <inertia ixx="0.083" ixy="0.0" ixz="0.0" iyy="0.083" iyz="0.0" izz="0.0"/>
     </inertial>
     <collision name="body">
-      <origin xyz="0.0 -.135 0.0"/>
+      <origin xyz="0 0 0"/>
       <geometry>
-        <box size="${width} ${length} ${height}"/>
+        <mesh filename="model://nautilus/meshes/nautilus_sim.dae"/>
       </geometry>
     </collision>
     <visual name="body">
       <geometry>
-        <mesh filename="model://nautilus/meshes/nautilus.dae"/>
+        <mesh filename="model://nautilus/meshes/nautilus_sim.dae"/>
       </geometry>
     </visual>

Commit message: Semi-stable, not balanced

File: src/nautilus_description/urdf/nautilus.urdf (robot description, URDF)
Before this commit: robot nautilus, 9 links, 8 joints
Links:
- link motor_A: mass 0.1658760921095411 -> 5.5; geometry collision mesh filename=model://nautilus/meshes/propeller.stl; visual mesh filename=model://nautilus/meshes/propeller.stl
- link motor_B: mass 0.1658760921095411 -> 5.5; geometry collision mesh filename=model://nautilus/meshes/propeller.stl; visual mesh filename=model://nautilus/meshes/propeller.stl
- link motor_C: mass 0.1658760921095411 -> 5.5; geometry collision mesh filename=model://nautilus/meshes/propeller.stl; visual mesh filename=model://nautilus/meshes/propeller.stl
- link motor_D: mass 0.1658760921095411 -> 5.5; geometry collision mesh filename=model://nautilus/meshes/propeller.stl; visual mesh filename=model://nautilus/meshes/propeller.stl
- link motor_E: mass 0.1658760921095411 -> 5.5; geometry collision mesh filename=model://nautilus/meshes/propeller.stl; visual mesh filename=model://nautilus/meshes/propeller.stl
- link motor_F: mass 0.1658760921095411 -> 5.5; geometry collision mesh filename=model://nautilus/meshes/propeller.stl; visual mesh filename=model://nautilus/meshes/propeller.stl
Joints:
- joint motor_A_joint: origin xyz=0.16 -0.34 -0.02 rpy=1.5707963267948966 0.0 -0.7853981633974483 -> xyz=0.259086 -0.00382228 0 rpy=1.5707963267948966 0.0 -0.7853981633974483
- joint motor_E_joint: origin xyz=0.165 -0.135 -0.02 rpy=0.0 0.0 0.0 -> xyz=0.259086 -0.00382228 0 rpy=0.0 0.0 0.0
- joint motor_F_joint: origin xyz=-0.165 -0.135 -0.02 rpy=0.0 0.0 0.0 -> xyz=-0.259691 -0.000494239 -0.02 rpy=0.0 0.0 0.0

File: src/nautilus_description/urdf/nautilus.urdf.xacro (robot description, xacro)
@@ -1,4 +1,5 @@
 <?xml version="1.0"?>
-<robot name="nautilus" xmlns:xacro="http://www.ros.org/wiki/xacro">
+<robot name="nautilus"
+  xmlns:xacro="http://www.ros.org/wiki/xacro">
   <!-- Constants -->
   <xacro:property name="PI" value="3.1415926535897931"/>
@@ -15,5 +16,5 @@
       <!-- TOOD: get a better mass estimate -->
       <mass value="60.177"/>
-     <inertia ixx="0.083" ixy="0.0" ixz="0.0" iyy="0.083" iyz="0.0" izz="0.0"/>
+      <inertia ixx="0.083" ixy="0.0" ixz="0.0" iyy="0.083" iyz="0.0" izz="0.0"/>
     </inertial>
     <collision name="body">
@@ -33,15 +34,15 @@
     <link name="${thrusterName}">
       <inertial>
-        <mass value="${PI * thruster_radius * thruster_radius * thruster_height * 1000}"/>
+        <mass value="5.5"/>
         <inertia ixx="0.4" ixy="0.0" ixz="0.0" iyy="0.4" iyz="0.0" izz="0.2"/>
       </inertial>
       <collision name="${thrusterName}">
         <geometry>
-          <cylinder radius="${thruster_radius}" length="${thruster_height}"/>
+          <mesh filename="model://nautilus/meshes/propeller.stl"/>
         </geometry>
       </collision>
       <visual name="${thrusterName}">
         <geometry>
-          <cylinder radius="${thruster_radius}" length="${thruster_height}"/>
+          <mesh filename="model://nautilus/meshes/propeller.stl"/>
         </geometry>
       </visual>
@@ -81,10 +82,10 @@
   <!-- y+ -> back -->
   <!-- z+ -> up -->
-  <xacro:thrusters thrusterName="motor_A" x=".16" y="-.34" z="-.02" r="${pi/2}" p="0.0" yaw="-${pi/4}"/>
+  <xacro:thrusters thrusterName="motor_A" x=".259086" y="-.00382228" z="0" r="${pi/2}" p="0.0" yaw="-${pi/4}"/>
   <xacro:thrusters thrusterName="motor_B" x="-.16" y="-.34" z="-.02" r="${pi/2}" p="0.0" yaw="${pi/4}"/>
   <xacro:thrusters thrusterName="motor_C" x=".16" y=".07" z="-.02" r="${pi/2}" p="0.0" yaw="${pi/4}"/>
   <xacro:thrusters thrusterName="motor_D" x="-.16" y=".07" z="-.02" r="${pi/2}" p="0.0" yaw="-${pi/4}"/>
-  <xacro:thrusters thrusterName="motor_E" x=".165" y="-.135" z="-.02" r="0.0" p="0.0" yaw="0.0"/>
-  <xacro:thrusters thrusterName="motor_F" x="-.165" y="-.135" z="-.02" r="0.0" p="0.0" yaw="0.0"/>
+  <xacro:thrusters thrusterName="motor_E" x=".259086" y="-.00382228" z="0" r="0.0" p="0.0" yaw="0.0"/>
+  <xacro:thrusters thrusterName="motor_F" x="-.259691" y="-.000494239" z="-.02" r="0.0" p="0.0" yaw="0.0"/>
   <xacro:cameras cameraName="camera1" x="0.0" y="-0.32" z="0.0" r="0.0" p="0.0" yaw="0.0"/>
   <xacro:cameras cameraName="camera2" x="0.0" y="-0.20" z="-.125" r="0.0" p="0.0" yaw="0.0"/>
