Commit message: Front thrusters

File: src/nautilus_description/urdf/rov22.urdf (robot description, URDF)
Before this commit: robot nautilus, 9 links, 8 joints
Links:
- link motor_A: mass 0.1658760921095411 -> 0.20993692907613795; geometry collision cylinder length=0.033 radius=0.045; visual cylinder length=0.033 radius=0.045
- link motor_B: mass 0.1658760921095411 -> 0.20993692907613795; geometry collision cylinder length=0.033 radius=0.045; visual cylinder length=0.033 radius=0.045
- link motor_C: mass 0.1658760921095411 -> 0.20993692907613795; geometry collision cylinder length=0.033 radius=0.045; visual cylinder length=0.033 radius=0.045
- link motor_D: mass 0.1658760921095411 -> 0.20993692907613795; geometry collision cylinder length=0.033 radius=0.045; visual cylinder length=0.033 radius=0.045
- link motor_E: mass 0.1658760921095411 -> 0.20993692907613795; geometry collision cylinder length=0.033 radius=0.045; visual cylinder length=0.033 radius=0.045
- link motor_F: mass 0.1658760921095411 -> 0.20993692907613795; geometry collision cylinder length=0.033 radius=0.045; visual cylinder length=0.033 radius=0.045
Joints:
- joint motor_A_joint: origin xyz=0.16 -0.34 -0.02 rpy=1.5707963267948966 0.0 -0.7853981633974483 -> xyz=0.1475 -0.283 -0.044 rpy=1.5707963267948966 0.0 0
- joint motor_B_joint: origin xyz=-0.16 -0.34 -0.02 rpy=1.5707963267948966 0.0 0.7853981633974483 -> xyz=-0.1475 -0.283 -0.044 rpy=1.5707963267948966 0.0 0

File: src/nautilus_description/urdf/rov22.urdf.xacro (robot description, xacro)
@@ -1,4 +1,5 @@
 <?xml version="1.0"?>
-<robot name="nautilus" xmlns:xacro="http://www.ros.org/wiki/xacro">
+<robot name="nautilus"
+  xmlns:xacro="http://www.ros.org/wiki/xacro">
   <!-- Constants -->
   <xacro:property name="PI" value="3.1415926535897931"/>
@@ -7,5 +8,5 @@
   <xacro:property name="length" value=".31"/>
   <xacro:property name="height" value=".24"/>
-  <xacro:property name="thruster_radius" value=".04"/>
+  <xacro:property name="thruster_radius" value=".045"/>
   <xacro:property name="thruster_height" value=".033"/>
   <!-- Begin defining the ROV -->
@@ -15,5 +16,5 @@
       <!-- TOOD: get a better mass estimate -->
       <mass value="21.576"/>
-     <inertia ixx="0.083" ixy="0.0" ixz="0.0" iyy="0.083" iyz="0.0" izz="0.0"/>
+      <inertia ixx="0.083" ixy="0.0" ixz="0.0" iyy="0.083" iyz="0.0" izz="0.0"/>
     </inertial>
     <collision name="body">
@@ -81,6 +82,6 @@
   <!-- y+ -> back -->
   <!-- z+ -> up -->
-  <xacro:thrusters thrusterName="motor_A" x=".16" y="-.34" z="-.02" r="${pi/2}" p="0.0" yaw="-${pi/4}"/>
-  <xacro:thrusters thrusterName="motor_B" x="-.16" y="-.34" z="-.02" r="${pi/2}" p="0.0" yaw="${pi/4}"/>
+  <xacro:thrusters thrusterName="motor_A" x=".1475" y="-.283" z="-.044" r="${pi/2}" p="0.0" yaw="0"/>
+  <xacro:thrusters thrusterName="motor_B" x="-.1475" y="-.283" z="-.044" r="${pi/2}" p="0.0" yaw="0"/>
   <xacro:thrusters thrusterName="motor_C" x=".16" y=".07" z="-.02" r="${pi/2}" p="0.0" yaw="${pi/4}"/>
   <xacro:thrusters thrusterName="motor_D" x="-.16" y=".07" z="-.02" r="${pi/2}" p="0.0" yaw="-${pi/4}"/>

Commit message: Vertical thrusters

File: src/nautilus_description/urdf/rov22.urdf (robot description, URDF)
Before this commit: robot nautilus, 9 links, 8 joints
Joints:
- joint motor_E_joint: origin xyz=0.165 -0.135 -0.02 rpy=0.0 0.0 0.0 -> xyz=0.1475 -0.135 0.044 rpy=0.0 0.0 0.0
- joint motor_F_joint: origin xyz=-0.165 -0.135 -0.02 rpy=0.0 0.0 0.0 -> xyz=-0.1475 -0.135 0.044 rpy=0.0 0.0 0.0

File: src/nautilus_description/urdf/rov22.urdf.xacro (robot description, xacro)
@@ -82,10 +82,14 @@
   <!-- y+ -> back -->
   <!-- z+ -> up -->
+  <!-- Port Bow -->
   <xacro:thrusters thrusterName="motor_A" x=".1475" y="-.283" z="-.044" r="${pi/2}" p="0.0" yaw="0"/>
+  <!-- Starboard Bow -->
   <xacro:thrusters thrusterName="motor_B" x="-.1475" y="-.283" z="-.044" r="${pi/2}" p="0.0" yaw="0"/>
   <xacro:thrusters thrusterName="motor_C" x=".16" y=".07" z="-.02" r="${pi/2}" p="0.0" yaw="${pi/4}"/>
   <xacro:thrusters thrusterName="motor_D" x="-.16" y=".07" z="-.02" r="${pi/2}" p="0.0" yaw="-${pi/4}"/>
-  <xacro:thrusters thrusterName="motor_E" x=".165" y="-.135" z="-.02" r="0.0" p="0.0" yaw="0.0"/>
-  <xacro:thrusters thrusterName="motor_F" x="-.165" y="-.135" z="-.02" r="0.0" p="0.0" yaw="0.0"/>
+  <!-- Port -->
+  <xacro:thrusters thrusterName="motor_E" x=".1475" y="-.135" z=".044" r="0.0" p="0.0" yaw="0.0"/>
+  <!-- Starboard -->
+  <xacro:thrusters thrusterName="motor_F" x="-.1475" y="-.135" z=".044" r="0.0" p="0.0" yaw="0.0"/>
   <xacro:cameras cameraName="camera1" x="0.0" y="-0.32" z="0.0" r="0.0" p="0.0" yaw="0.0"/>
   <xacro:cameras cameraName="camera2" x="0.0" y="-0.20" z="-.125" r="0.0" p="0.0" yaw="0.0"/>

Commit message: Bow Thruster

File: src/nautilus_description/urdf/rov22.urdf (robot description, URDF)
Before this commit: robot nautilus, 9 links, 8 joints
Joints:
- joint motor_C_joint: origin xyz=0.16 0.07 -0.02 rpy=1.5707963267948966 0.0 0.7853981633974483 -> xyz=0 -0.331 0.15 rpy=0 1.5707963267948966 0

File: src/nautilus_description/urdf/rov22.urdf.xacro (robot description, xacro)
@@ -86,10 +86,12 @@
   <!-- Starboard Bow -->
   <xacro:thrusters thrusterName="motor_B" x="-.1475" y="-.283" z="-.044" r="${pi/2}" p="0.0" yaw="0"/>
-  <xacro:thrusters thrusterName="motor_C" x=".16" y=".07" z="-.02" r="${pi/2}" p="0.0" yaw="${pi/4}"/>
-  <xacro:thrusters thrusterName="motor_D" x="-.16" y=".07" z="-.02" r="${pi/2}" p="0.0" yaw="-${pi/4}"/>
   <!-- Port -->
   <xacro:thrusters thrusterName="motor_E" x=".1475" y="-.135" z=".044" r="0.0" p="0.0" yaw="0.0"/>
   <!-- Starboard -->
   <xacro:thrusters thrusterName="motor_F" x="-.1475" y="-.135" z=".044" r="0.0" p="0.0" yaw="0.0"/>
+  <!-- Bow -->
+  <xacro:thrusters thrusterName="motor_C" x="0" y="-.331" z=".15" r="0" p="${pi/2}" yaw="0"/>
+  <!-- Stern -->
+  <xacro:thrusters thrusterName="motor_D" x="-.16" y=".07" z="-.02" r="${pi/2}" p="0.0" yaw="-${pi/4}"/>
   <xacro:cameras cameraName="camera1" x="0.0" y="-0.32" z="0.0" r="0.0" p="0.0" yaw="0.0"/>
   <xacro:cameras cameraName="camera2" x="0.0" y="-0.20" z="-.125" r="0.0" p="0.0" yaw="0.0"/>

Commit message: Stern Thruster

File: src/nautilus_description/urdf/rov22.urdf (robot description, URDF)
Before this commit: robot nautilus, 9 links, 8 joints
Joints:
- joint motor_D_joint: origin xyz=-0.16 0.07 -0.02 rpy=1.5707963267948966 0.0 -0.7853981633974483 -> xyz=0 -0.019 0.15 rpy=1.5707963267948966 0.0 0

File: src/nautilus_description/urdf/rov22.urdf.xacro (robot description, xacro)
@@ -93,5 +93,5 @@
   <xacro:thrusters thrusterName="motor_C" x="0" y="-.331" z=".15" r="0" p="${pi/2}" yaw="0"/>
   <!-- Stern -->
-  <xacro:thrusters thrusterName="motor_D" x="-.16" y=".07" z="-.02" r="${pi/2}" p="0.0" yaw="-${pi/4}"/>
+  <xacro:thrusters thrusterName="motor_D" x="0" y="-.019" z=".15" r="${pi/2}" p="0.0" yaw="0"/>
   <xacro:cameras cameraName="camera1" x="0.0" y="-0.32" z="0.0" r="0.0" p="0.0" yaw="0.0"/>
   <xacro:cameras cameraName="camera2" x="0.0" y="-0.20" z="-.125" r="0.0" p="0.0" yaw="0.0"/>

Commit message: More intuitive motor config, drive forward-ish

File: src/nautilus_description/urdf/rov22.urdf (robot description, URDF)
Before this commit: robot nautilus, 9 links, 8 joints
Joints:
- joint motor_D_joint: origin xyz=0 -0.019 0.15 rpy=1.5707963267948966 0.0 0 -> xyz=0.1475 -0.135 0.044 rpy=0.0 0.0 0.0
- joint motor_E_joint: origin xyz=0.1475 -0.135 0.044 rpy=0.0 0.0 0.0 -> xyz=-0.1475 -0.135 0.044 rpy=0.0 0.0 0.0
- joint motor_F_joint: origin xyz=-0.1475 -0.135 0.044 rpy=0.0 0.0 0.0 -> xyz=0 -0.019 0.15 rpy=1.5707963267948966 0.0 0

File: src/nautilus_description/urdf/rov22.urdf.xacro (robot description, xacro)
@@ -82,16 +82,16 @@
   <!-- y+ -> back -->
   <!-- z+ -> up -->
-  <!-- Port Bow -->
+  <!-- A: Port Bow -->
   <xacro:thrusters thrusterName="motor_A" x=".1475" y="-.283" z="-.044" r="${pi/2}" p="0.0" yaw="0"/>
-  <!-- Starboard Bow -->
+  <!-- B: Starboard Bow -->
   <xacro:thrusters thrusterName="motor_B" x="-.1475" y="-.283" z="-.044" r="${pi/2}" p="0.0" yaw="0"/>
-  <!-- Port -->
-  <xacro:thrusters thrusterName="motor_E" x=".1475" y="-.135" z=".044" r="0.0" p="0.0" yaw="0.0"/>
-  <!-- Starboard -->
-  <xacro:thrusters thrusterName="motor_F" x="-.1475" y="-.135" z=".044" r="0.0" p="0.0" yaw="0.0"/>
-  <!-- Bow -->
+  <!-- C: Bow -->
   <xacro:thrusters thrusterName="motor_C" x="0" y="-.331" z=".15" r="0" p="${pi/2}" yaw="0"/>
-  <!-- Stern -->
-  <xacro:thrusters thrusterName="motor_D" x="0" y="-.019" z=".15" r="${pi/2}" p="0.0" yaw="0"/>
+  <!-- D: Port -->
+  <xacro:thrusters thrusterName="motor_D" x=".1475" y="-.135" z=".044" r="0.0" p="0.0" yaw="0.0"/>
+  <!-- E: Starboard -->
+  <xacro:thrusters thrusterName="motor_E" x="-.1475" y="-.135" z=".044" r="0.0" p="0.0" yaw="0.0"/>
+  <!-- F: Stern -->
+  <xacro:thrusters thrusterName="motor_F" x="0" y="-.019" z=".15" r="${pi/2}" p="0.0" yaw="0"/>
   <xacro:cameras cameraName="camera1" x="0.0" y="-0.32" z="0.0" r="0.0" p="0.0" yaw="0.0"/>
   <xacro:cameras cameraName="camera2" x="0.0" y="-0.20" z="-.125" r="0.0" p="0.0" yaw="0.0"/>
